File: LEDMatrix.brd (EAGLE design)
At the start: 50 x 50 mm, 22 parts

Commit message: updated silk layer
Parts:
- added CC_TEXT1: CREATIVE_COMMONS, SparkFun-Aesthetics:CREATIVE_COMMONS
- added LOGO1: OSHW-LOGOL, SparkFun-Aesthetics:OSHW-LOGO-L
- SJ2: value LED_VDD -> Vdigital
Routing:
- net N$9: track 48.1 -> 46.9 mm
Other:
- board text added: "Vdigital"
- board text removed: "LED_VDD"

Commit message: replaced parts library (schematic only)
Parts:
- IC1: value (none) -> HT1632C
- renumbered X1 to IC1
Changed lines of the file:
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@@
 </autorouter>
 <elements>
-<element name="X1" library="HT1632" package="QFP52" value="" x="30.48" y="29.845" smashed="yes" rot="R180">
+<element name="IC1" library="HT1632" package="QFP52" value="HT1632C" x="30.48" y="29.845" smashed="yes" rot="R180">
 <attribute name="VALUE" x="37.465" y="20.32" size="1.27" layer="27" rot="R180"/>
 </element>
@@
 <signals>
 <signal name="COM7">
-<contactref element="X1" pad="P$30"/>
+<contactref element="IC1" pad="P$30"/>
 <contactref element="U$1" pad="1"/>
 <contactref element="SJ5" pad="1"/>
@@
 </signal>
 <signal name="COM0">
-<contactref element="X1" pad="P$22"/>
+<contactref element="IC1" pad="P$22"/>
 <contactref element="U$1" pad="8"/>
 <contactref element="SJ12" pad="1"/>
@@
 </signal>
 <signal name="COM1">
-<contactref element="X1" pad="P$23"/>
+<contactref element="IC1" pad="P$23"/>
 <contactref element="U$1" pad="7"/>
 <contactref element="SJ11" pad="1"/>
@@
 </signal>
 <signal name="COM2">
-<contactref element="X1" pad="P$24"/>
+<contactref element="IC1" pad="P$24"/>
 <contactref element="U$1" pad="6"/>
 <contactref element="SJ10" pad="1"/>
@@
 </signal>
 <signal name="COM3">
-<contactref element="X1" pad="P$26"/>
+<contactref element="IC1" pad="P$26"/>
 <contactref element="U$1" pad="5"/>
 <contactref element="SJ9" pad="1"/>
@@
 </signal>
 <signal name="COM4">
-<contactref element="X1" pad="P$27"/>
+<contactref element="IC1" pad="P$27"/>
 <contactref element="U$1" pad="4"/>
 <contactref element="SJ8" pad="1"/>
@@
 </signal>
 <signal name="COM5">
-<contactref element="X1" pad="P$28"/>
+<contactref element="IC1" pad="P$28"/>
 <contactref element="U$1" pad="3"/>
 <contactref element="SJ7" pad="1"/>
@@
 </signal>
 <signal name="COM6">
-<contactref element="X1" pad="P$29"/>
+<contactref element="IC1" pad="P$29"/>
 <contactref element="U$1" pad="2"/>
 <contactref element="SJ6" pad="1"/>
@@
 </signal>
 <signal name="GND">
-<contactref element="X1" pad="P$14"/>
-<contactref element="X1" pad="P$25"/>
-<contactref element="X1" pad="P$36"/>
+<contactref element="IC1" pad="P$14"/>
+<contactref element="IC1" pad="P$25"/>
+<contactref element="IC1" pad="P$36"/>
 <contactref element="SJ1" pad="3"/>
 <polygon width="0.254" layer="1" isolate="0.254">
@@
 </signal>
 <signal name="ROW2">
-<contactref element="X1" pad="P$11"/>
+<contactref element="IC1" pad="P$11"/>
 <contactref element="R1" pad="3"/>
 <wire x1="13.96" y1="44.85" x2="18.65" y2="44.85" width="0.254" layer="1"/>
@@
 </signal>
 <signal name="ROW0">
-<contactref element="X1" pad="P$13"/>
+<contactref element="IC1" pad="P$13"/>
 <contactref element="R1" pad="1"/>
 <wire x1="13.96" y1="43.25" x2="18.98" y2="43.25" width="0.254" layer="1"/>
@@
 </signal>
 <signal name="ROW1">
-<contactref element="X1" pad="P$12"/>
+<contactref element="IC1" pad="P$12"/>
 <contactref element="R1" pad="2"/>
 <wire x1="13.96" y1="44.05" x2="18.815" y2="44.05" width="0.254" layer="1"/>
@@
 </signal>
 <signal name="ROW3">
-<contactref element="X1" pad="P$10"/>
+<contactref element="IC1" pad="P$10"/>
 <contactref element="R1" pad="4"/>
 <wire x1="13.96" y1="45.65" x2="18.485" y2="45.65" width="0.254" layer="1"/>
@@
 </signal>
 <signal name="ROW4">
-<contactref element="X1" pad="P$9"/>
+<contactref element="IC1" pad="P$9"/>
 <contactref element="R2" pad="1"/>
 <wire x1="24.12" y1="43.25" x2="26.6" y2="43.25" width="0.254" layer="1"/>
@@
 </signal>
 <signal name="ROW5">
-<contactref element="X1" pad="P$8"/>
+<contactref element="IC1" pad="P$8"/>
 <contactref element="R2" pad="2"/>
 <wire x1="24.12" y1="44.05" x2="26.435" y2="44.05" width="0.254" layer="1"/>
@@
 </signal>
 <signal name="ROW6">
-<contactref element="X1" pad="P$6"/>
+<contactref element="IC1" pad="P$6"/>
 <contactref element="R2" pad="3"/>
 <wire x1="24.12" y1="44.85" x2="26.27" y2="44.85" width="0.254" layer="1"/>
@@
 </signal>
 <signal name="ROW7">
-<contactref element="X1" pad="P$5"/>
+<contactref element="IC1" pad="P$5"/>
 <contactref element="R2" pad="4"/>
 <wire x1="24.12" y1="45.65" x2="26.105" y2="45.65" width="0.254" layer="1"/>
@@
 </signal>
 <signal name="ROW8">
-<contactref element="X1" pad="P$4"/>
+<contactref element="IC1" pad="P$4"/>
 <contactref element="R3" pad="1"/>
 <wire x1="33.01" y1="43.25" x2="33.1625" y2="43.25" width="0.254" layer="1"/>
@@
 </signal>
 <signal name="ROW9">
-<contactref element="X1" pad="P$3"/>
+<contactref element="IC1" pad="P$3"/>
 <contactref element="R3" pad="2"/>
 <wire x1="33.01" y1="44.05" x2="34.055" y2="44.05" width="0.254" layer="1"/>
@@
 </signal>
 <signal name="ROW10">
-<contactref element="X1" pad="P$2"/>
+<contactref element="IC1" pad="P$2"/>
 <contactref element="R3" pad="3"/>
 <wire x1="33.01" y1="44.85" x2="34.525" y2="44.85" width="0.254" layer="1"/>
@@
 </signal>
 <signal name="ROW11">
-<contactref element="X1" pad="P$1"/>
+<contactref element="IC1" pad="P$1"/>
 <contactref element="R3" pad="4"/>
 <wire x1="33.01" y1="45.65" x2="34.995" y2="45.65" width="0.254" layer="1"/>
@@
 </signal>
 <signal name="ROW12">
-<contactref element="X1" pad="P$52"/>
+<contactref element="IC1" pad="P$52"/>
 <contactref element="R4" pad="1"/>
 <wire x1="38.805" y1="43.19" x2="38.805" y2="35.97" width="0.254" layer="1"/>
@@
 </signal>
 <signal name="ROW13">
-<contactref element="X1" pad="P$51"/>
+<contactref element="IC1" pad="P$51"/>
 <contactref element="R4" pad="2"/>
 <wire x1="39.605" y1="43.19" x2="39.605" y2="42.31" width="0.254" layer="1"/>
@@
 </signal>
 <signal name="ROW14">
-<contactref element="X1" pad="P$50"/>
+<contactref element="IC1" pad="P$50"/>
 <contactref element="R4" pad="3"/>
 <wire x1="40.405" y1="43.19" x2="40.405" y2="42.78" width="0.254" layer="1"/>
@@
 </signal>
 <signal name="ROW15">
-<contactref element="X1" pad="P$49"/>
+<contactref element="IC1" pad="P$49"/>
 <contactref element="R4" pad="4"/>
 <wire x1="41.205" y1="43.19" x2="41.205" y2="43.25" width="0.254" layer="1"/>
@@
 </signal>
 <signal name="ROW16">
-<contactref element="X1" pad="P$48"/>
+<contactref element="IC1" pad="P$48"/>
 <contactref element="R6" pad="5"/>
 <wire x1="38.68" y1="31.845" x2="45.9675" y2="31.845" width="0.254" layer="1"/>
@@
 </signal>
 <signal name="ROW17">
-<contactref element="X1" pad="P$47"/>
+<contactref element="IC1" pad="P$47"/>
 <contactref element="R6" pad="6"/>
 <wire x1="38.68" y1="30.845" x2="45.1675" y2="30.845" width="0.254" layer="1"/>
@@
 </signal>
 <signal name="ROW18">
-<contactref element="X1" pad="P$46"/>
+<contactref element="IC1" pad="P$46"/>
 <contactref element="R6" pad="7"/>
 <wire x1="38.68" y1="29.845" x2="44.3675" y2="29.845" width="0.254" layer="1"/>
@@
 </signal>
 <signal name="ROW19">
-<contactref element="X1" pad="P$45"/>
+<contactref element="IC1" pad="P$45"/>
 <contactref element="R6" pad="8"/>
 <wire x1="38.68" y1="28.845" x2="43.5675" y2="28.845" width="0.254" layer="1"/>
@@
 </signal>
 <signal name="ROW20">
-<contactref element="X1" pad="P$44"/>
+<contactref element="IC1" pad="P$44"/>
 <contactref element="R5" pad="5"/>
 <wire x1="38.68" y1="27.845" x2="42.1575" y2="27.845" width="0.254" layer="1"/>
@@
 </signal>
 <signal name="ROW21">
-<contactref element="X1" pad="P$43"/>
+<contactref element="IC1" pad="P$43"/>
 <contactref element="R5" pad="6"/>
 <wire x1="38.68" y1="26.845" x2="41.3575" y2="26.845" width="0.254" layer="1"/>
@@
 </signal>
 <signal name="ROW22">
-<contactref element="X1" pad="P$42"/>
+<contactref element="IC1" pad="P$42"/>
 <contactref element="R5" pad="7"/>
 <wire x1="38.68" y1="25.845" x2="40.5575" y2="25.845" width="0.254" layer="1"/>
@@
 </signal>
 <signal name="ROW23">
-<contactref element="X1" pad="P$41"/>
+<contactref element="IC1" pad="P$41"/>
 <contactref element="R5" pad="8"/>
 <wire x1="38.68" y1="24.845" x2="39.7575" y2="24.845" width="0.254" layer="1"/>
@@
 </signal>
 <signal name="!CS">
-<contactref element="X1" pad="P$19"/>
+<contactref element="IC1" pad="P$19"/>
 <wire x1="22.28" y1="30.845" x2="19.415" y2="30.845" width="0.254" layer="1"/>
 <wire x1="19.415" y1="30.845" x2="15.875" y2="27.305" width="0.254" layer="1"/>
@@
 </signal>
 <signal name="!RD">
-<contactref element="X1" pad="P$18"/>
+<contactref element="IC1" pad="P$18"/>
 <wire x1="22.28" y1="31.845" x2="19.145" y2="31.845" width="0.254" layer="1"/>
 <wire x1="19.145" y1="31.845" x2="15.24" y2="27.94" width="0.254" layer="1"/>
@@
 </signal>
 <signal name="!WR">
-<contactref element="X1" pad="P$17"/>
+<contactref element="IC1" pad="P$17"/>
 <wire x1="22.28" y1="32.845" x2="18.875" y2="32.845" width="0.254" layer="1"/>
 <wire x1="18.875" y1="32.845" x2="13.97" y2="27.94" width="0.254" layer="1"/>
@@
 </signal>
 <signal name="DATA">
-<contactref element="X1" pad="P$16"/>
+<contactref element="IC1" pad="P$16"/>
 <wire x1="22.28" y1="33.845" x2="18.605" y2="33.845" width="0.254" layer="1"/>
 <wire x1="18.605" y1="33.845" x2="15.24" y2="30.48" width="0.254" layer="1"/>
@@
 </signal>
 <signal name="OSC">
-<contactref element="X1" pad="P$15"/>
+<contactref element="IC1" pad="P$15"/>
 <contactref element="SJ1" pad="2"/>
 <wire x1="22.28" y1="34.845" x2="18.335" y2="34.845" width="0.254" layer="1"/>
@@
 </signal>
 <signal name="SYNC">
-<contactref element="X1" pad="P$20"/>
+<contactref element="IC1" pad="P$20"/>
 <wire x1="22.28" y1="29.845" x2="19.685" y2="29.845" width="0.254" layer="1"/>
 <wire x1="19.685" y1="29.845" x2="16.51" y2="26.67" width="0.254" layer="1"/>
@@
 <contactref element="SJ3" pad="3"/>
 <contactref element="JP2" pad="6"/>
-<contactref element="X1" pad="P$38"/>
-<contactref element="X1" pad="P$7"/>
+<contactref element="IC1" pad="P$38"/>
+<contactref element="IC1" pad="P$7"/>
 <wire x1="30.48" y1="37.945" x2="30.48" y2="33.02" width="0.4064" layer="1"/>
 <via x="30.48" y="33.02" extent="1-16" drill="0.6" shape="octagon"/>
@@
 </signal>
 <signal name="N$9">
-<contactref element="X1" pad="P$21"/>
+<contactref element="IC1" pad="P$21"/>
 <contactref element="SJ2" pad="2"/>
 <via x="37.465" y="15.24" extent="1-16" drill="0.6" shape="octagon"/>
